File: JSerial2g.sch (EAGLE design)
At the start: 59 parts, among them CN1 USBMOLEX, IC1 FT232RL, Q1 2N3904SOT23, Q2 2N3904SOT23, Q3 BC547, Q4 BC547, X1 RJ45-8X

Commit message: JSerial 2G in progress
Parts:
- removed C3: 0.47 uF, ipc-7351-capacitor:CAPACITOR_0805
- removed J1, J4: (no value), jlab:POWER-OUT
- removed JP10, JP11, JP12, JP13, JP14, JP15, JP16, JP17, JP18, JP19, JP20, JP21, JP22, JP23, JP24, JP25, JP26, JP27, JP28, JP35, JP4, JP5, JP6, JP7, JP9: (no value), pinhead:PINHD-1X1
- removed JP29: (no value), pinhead:PINHD-2X10
- removed JP3: (no value), pinhead:PINHD-2X12
- removed JP30: (no value), pinhead:PINHD-2X6
- removed JP8: (no value), pinhead:PINHD-1X7
- removed Q2: 2N3904SOT23, transistor-npn:2N3904SOT23
- removed Q3, Q4: BC547, transistor-npn:BC547
- removed S1: DT5X6, jlab:DT5X6
- added C4, C5, C6, C7: 0.1uF, ipc-7351-capacitor:CAPACITOR_0805
- added D1: 1N4148, diode:DIODE-SOD123
- added IC2: MAX3232CSE, maxim:MAX3232CSE
- added J2: DCJ0202, con-jack:DCJ0202
- added Q5, Q6, Q8: BC857BSMD, transistor-pnp:BC857BSMD
- added Q9: 2N3904SOT23, transistor-npn:2N3904SOT23
- added R10, R12, R14: 1K, ipc-7351-resistor:RESISTOR_0805
- added R11, R13, R9: 10K, ipc-7351-resistor:RESISTOR_0805
- added R15: 100, ipc-7351-resistor:RESISTOR_0805
- added R8: 4.7K, ipc-7351-resistor:RESISTOR_0805
- added SP1: KSS1201, buzzer:KSS1201
- added X2: (no value), jlab:M09D
- JP1: device pinhead:PINHD-2X6 -> pinhead:PINHD-1X1
- JP2: device pinhead:PINHD-2X12 -> pinhead:PINHD-1X1
- LED2, LED3: device jlab:LEDCHIP-LED0805 -> jlab:LED3MM
- R2, R3: value 270 R -> 470
- R4, R7: value 270 R -> 1K
- R5, R6: value 270 R -> 10K
Connections:
- net RT renamed RI
- removed net N$23: JP22.1, R4.1
- removed net N$24: JP14.1, Q3.C
- removed net N$25: JP18.1, Q4.C
- removed net N$26: JP19.1, Q4.E
- removed net N$27: JP20.1, Q3.E
- removed net N$28: JP23.1, R5.1
- removed net N$29: JP24.1, R7.1
- removed net N$30: JP13.1, Q1.C
- removed net N$31: JP15.1, Q1.E
- removed net N$32: JP17.1, Q2.C
- removed net N$33: JP16.1, Q2.E
- removed net N$34: JP25.1, R7.2
- removed net N$35: JP26.1, R5.2
- removed net N$36: JP27.1, R4.2
- removed net N$37: JP28.1, R6.2
- removed net OSCO: IC1.OSCO, JP8.2
- new net N$13: IC2G$1.R1IN, X2.2
- new net N$14: J2.1, Q8.C
- new net N$15: Q5.B, R5.1, R7.2
- new net N$16: Q6.B, R4.2, R6.1
- new net N$17: Q9.B, R10.2, R11.2
- new net N$2: C4.1, IC2G$1.C1-
- new net N$7: C4.2, IC2G$1.C1+
- new net N$8: C5.1, IC2G$1.C2-
- new net TX_TTL_INV: IC1.RXD, Q5.C, Q6.C, R8.2
- new net TX_TTL_MAXIM: IC2G$1.R1OUT, R4.1
- net +3V3: now also C6.2, IC2P.VCC, Q5.E, Q6.E, R13.2, R5.2, R6.2; no longer JP3.10, JP3.12, JP3.14, JP3.16, JP3.18, JP3.2, JP3.20, JP3.22, JP3.24, JP3.4, JP3.6, JP3.8
- net +5V: now also Q8.E, R15.2, R9.2; no longer JP29.10, JP29.12, JP29.14, JP29.16, JP29.18, JP29.2, JP29.20, JP29.4, JP29.6, JP29.8
- net CBUS0: no longer JP8.1
- net CBUS2: now also R10.1; no longer JP8.6
- net CBUS3: now also JP33.1; no longer JP8.7
- net CBUS4: now also JP2.1; no longer JP8.5
- net DCD: now also J2.2, R13.1; no longer JP33.1
- net DTR: now also JP1.1; no longer JP8.4
- net GND: now also C7.2, IC2P.GND, J2.3, Q1.E, Q9.E, R11.1, R8.1, X2.5; no longer C3.1, JP2.10, JP2.12, JP2.14, JP2.16, JP2.18, JP2.2, JP2.20, JP2.22, JP2.24, JP2.4, JP2.6, JP2.8
- net N$10: now also C6.1, IC2G$1.V+; no longer J1GND.P$1, JP5.1
- net N$11: now also C7.1, IC2G$1.V-; no longer J4PLUS.P$1, JP6.1
- net N$12: now also IC2G$1.T1OUT, X2.3; no longer J4GND.P$1, JP7.1
- net N$18: now also Q9.C, R12.1; no longer JP9.1, Q3.B
- net N$19: now also Q8.B, R12.2, R9.1; no longer JP10.1, Q4.B
- net N$20: now also Q1.B, R14.2; no longer JP12.1, Q2.B
- net N$21: now also D1.A, Q1.C, SP1.2; no longer JP11.1, Q1.B
- net N$22: now also D1.C, R15.1, SP1.1; no longer JP21.1, R6.1
- net N$9: now also C5.2, IC2G$1.C2+; no longer J1PLUS.P$1, JP4.1
- net RTS: now also R14.1; no longer JP8.3
- net RX_TTL: now also IC2G$1.T1IN
- net TX_TTL: now also R7.1; no longer IC1.RXD
- net VCC: no longer C3.2, JP35.1
Other:
- moved on the sheet: C1, C11, C2, CN1, IC1, JP31, JP32, JP33, JP34, LED1, LED2, LED3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

Commit message: Work in progress
Parts:
- added C3: 0.1 uF, ipc-7351-capacitor:CAPACITOR_0805
- D1: device diode:DIODE-SOD123 -> ipc-7351-diode:DIODE_SOD-123
- LED1: device jlab:LEDCHIP-LED0805 -> jlab:LED3MM
- Q1: value 2N3904SOT23 -> 2N3904 SOT23; device transistor-npn:2N3904SOT23 -> ipc-7351-transistor:NPN_SOT-23
- Q9: value 2N3904SOT23 -> 2N3904; device transistor-npn:2N3904SOT23 -> ipc-7351-transistor:NPN_SOT-23
Connections:
- net +3V3: now also C3.2
- net GND: now also C3.1
- net N$22: now also D1.K; no longer D1.C
Changed lines of the file:
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@@
 <part name="C2" library="ipc-7351-capacitor" deviceset="CAPACITOR_" device="0805" value="0.47 uF"/>
 <part name="R1" library="ipc-7351-resistor" deviceset="RESISTOR_" device="0805" value="270 R"/>
-<part name="LED1" library="jlab" deviceset="LED" device="CHIP-LED0805" value="Green"/>
+<part name="LED1" library="jlab" deviceset="LED" device="3MM" value="Green"/>
 <part name="GND1" library="supply1" deviceset="GND" device=""/>
 <part name="+3V2" library="supply1" deviceset="VCC" device=""/>
@@
 <part name="Q6" library="transistor-pnp" deviceset="BC857*" device="SMD" technology="B"/>
 <part name="Q8" library="transistor-pnp" deviceset="BC857*" device="SMD" technology="B"/>
-<part name="Q9" library="transistor-npn" deviceset="2N3904" device="SOT23"/>
-<part name="D1" library="diode" deviceset="DIODE-" device="SOD123" value="1N4148"/>
+<part name="Q9" library="ipc-7351-transistor" deviceset="NPN_" device="SOT-23" value="2N3904"/>
+<part name="D1" library="ipc-7351-diode" deviceset="DIODE_" device="SOD-123" value="1N4148"/>
 <part name="SP1" library="buzzer" deviceset="KSS1201" device=""/>
 <part name="GND10" library="supply1" deviceset="GND" device=""/>
@@
 <part name="+3V5" library="supply1" deviceset="+3V3" device=""/>
 <part name="R13" library="ipc-7351-resistor" deviceset="RESISTOR_" device="0805" value="10K"/>
-<part name="Q1" library="transistor-npn" deviceset="2N3904" device="SOT23"/>
+<part name="Q1" library="ipc-7351-transistor" deviceset="NPN_" device="SOT-23" value="2N3904 SOT23"/>
 <part name="P+6" library="supply1" deviceset="+5V" device=""/>
 <part name="R14" library="ipc-7351-resistor" deviceset="RESISTOR_" device="0805" value="1K"/>
@@
 <part name="JP1" library="pinhead" deviceset="PINHD-1X1" device=""/>
 <part name="JP2" library="pinhead" deviceset="PINHD-1X1" device=""/>
+<part name="C3" library="ipc-7351-capacitor" deviceset="CAPACITOR_" device="0805" value="0.1 uF"/>
+<part name="GND18" library="supply1" deviceset="GND" device=""/>
+<part name="+3V11" library="supply1" deviceset="+3V3" device=""/>
 </parts>
 <sheets>
@@
 <instance part="Q6" gate="G$1" x="160.02" y="71.12"/>
 <instance part="Q8" gate="G$1" x="302.26" y="99.06"/>
-<instance part="Q9" gate="G1" x="264.16" y="93.98"/>
+<instance part="Q9" gate="G$1" x="264.16" y="93.98"/>
 <instance part="D1" gate="G$1" x="312.42" y="215.9" rot="R90"/>
 <instance part="SP1" gate="1" x="322.58" y="215.9" rot="R270"/>
@@
 <instance part="+3V5" gate="G$1" x="322.58" y="114.3" rot="MR0"/>
 <instance part="R13" gate="G$1" x="322.58" y="106.68" rot="R90"/>
-<instance part="Q1" gate="G1" x="320.04" y="198.12"/>
+<instance part="Q1" gate="G$1" x="320.04" y="198.12"/>
 <instance part="P+6" gate="1" x="322.58" y="241.3"/>
 <instance part="R14" gate="G$1" x="302.26" y="198.12"/>
@@
 <instance part="JP1" gate="G$1" x="170.18" y="231.14"/>
 <instance part="JP2" gate="G$1" x="195.58" y="190.5"/>
+<instance part="C3" gate="G$1" x="43.18" y="25.4" rot="R90"/>
+<instance part="GND18" gate="1" x="43.18" y="15.24"/>
+<instance part="+3V11" gate="G$1" x="43.18" y="40.64"/>
 </instances>
 <busses>
@@
 <segment>
 <pinref part="GND15" gate="1" pin="GND"/>
-<pinref part="Q9" gate="G1" pin="E"/>
+<pinref part="Q9" gate="G$1" pin="E"/>
 <wire x1="266.7" y1="76.2" x2="266.7" y2="88.9" width="0.1524" layer="91"/>
 </segment>
@@
 </segment>
 <segment>
-<pinref part="Q1" gate="G1" pin="E"/>
+<pinref part="Q1" gate="G$1" pin="E"/>
 <pinref part="GND17" gate="1" pin="GND"/>
 <wire x1="322.58" y1="185.42" x2="322.58" y2="193.04" width="0.1524" layer="91"/>
+</segment>
+<segment>
+<pinref part="GND18" gate="1" pin="GND"/>
+<pinref part="C3" gate="G$1" pin="1"/>
+<wire x1="43.18" y1="17.78" x2="43.18" y2="20.32" width="0.1524" layer="91"/>
 </segment>
 </net>
@@
 <pinref part="R13" gate="G$1" pin="2"/>
 </segment>
+<segment>
+<pinref part="C3" gate="G$1" pin="2"/>
+<pinref part="+3V11" gate="G$1" pin="+3V3"/>
+<wire x1="43.18" y1="38.1" x2="43.18" y2="30.48" width="0.1524" layer="91"/>
+</segment>
 </net>
 <net name="N$2" class="0">
@@
 <segment>
 <pinref part="R10" gate="G$1" pin="2"/>
-<pinref part="Q9" gate="G1" pin="B"/>
+<pinref part="Q9" gate="G$1" pin="B"/>
 <wire x1="248.92" y1="93.98" x2="256.54" y2="93.98" width="0.1524" layer="91"/>
 <pinref part="R11" gate="G$1" pin="2"/>
@@
 <net name="N$18" class="0">
 <segment>
-<pinref part="Q9" gate="G1" pin="C"/>
+<pinref part="Q9" gate="G$1" pin="C"/>
 <pinref part="R12" gate="G$1" pin="1"/>
 <wire x1="266.7" y1="99.06" x2="269.24" y2="99.06" width="0.1524" layer="91"/>
@@
 <net name="N$20" class="0">
 <segment>
-<pinref part="Q1" gate="G1" pin="B"/>
+<pinref part="Q1" gate="G$1" pin="B"/>
 <pinref part="R14" gate="G$1" pin="2"/>
 <wire x1="307.34" y1="198.12" x2="317.5" y2="198.12" width="0.1524" layer="91"/>
@@
 <net name="N$21" class="0">
 <segment>
-<pinref part="Q1" gate="G1" pin="C"/>
+<pinref part="Q1" gate="G$1" pin="C"/>
 <pinref part="SP1" gate="1" pin="2"/>
 <wire x1="322.58" y1="210.82" x2="322.58" y2="208.28" width="0.1524" layer="91"/>
@@
 <pinref part="R15" gate="G$1" pin="1"/>
 <wire x1="322.58" y1="223.52" x2="322.58" y2="220.98" width="0.1524" layer="91"/>
-<pinref part="D1" gate="G$1" pin="C"/>
+<pinref part="D1" gate="G$1" pin="K"/>
 <wire x1="312.42" y1="218.44" x2="312.42" y2="223.52" width="0.1524" layer="91"/>
 <wire x1="312.42" y1="223.52" x2="322.58" y2="223.52" width="0.1524" layer="91"/>

Commit message: layout finished. start review
Parts:
- removed C11: 10uF, ipc-7351-capacitor:POLARISED_A_CASE
- removed X2: (no value), jlab:M09D
- added C8, C9: 0.1uF, ipc-7351-capacitor:CAPACITOR_0805
- added J1: DCJ0202, con-jack:DCJ0202
- C1: value 0.47 uF -> 0.1 uF
- C3: value 0.1 uF -> 10uF; device ipc-7351-capacitor:CAPACITOR_0805 -> ipc-7351-capacitor:POLARISED_A_CASE
- C4: value 0.1uF -> 100uF; device ipc-7351-capacitor:CAPACITOR_0805 -> rcl:CPOL-EUE2.5-6
- C5: value 0.1uF -> 0.47 uF
- CB0, CB1, LED1: value Green -> (none)
- J2: value DCJ0202 -> (none); device con-jack:DCJ0202 -> jlab:M09D
- R1: value 270 R -> 1K
- R2, R3: value 470 -> 1K
- R6: value 10K -> 4.7K
- R8: value 4.7K -> 10K
- renumbered CN1 to J4, JP1 to DTR, JP2 to CB4, JP31 to CTS, JP32 to DSR, JP33 to CB3, JP34 to RI, LED2 to CB0, LED3 to CB1, X1 to J3
Connections:
- net +3V3: now also C5.2, R8.2; no longer C3.2, R6.2
- net +5V: now also C3.+, C4.+; no longer C11.+
- net DCD: now also J1.2; no longer J2.2
- net GND: now also C3.-, C4.-, C5.1, J1.3, J2.5, R6.1; no longer C11.-, C3.1, J2.3, R8.1, X2.5
- net N$12: now also J2.3; no longer X2.3
- net N$13: now also J2.2; no longer X2.2
- net N$14: now also J1.1; no longer J2.1
- net N$15: now also R4.2; no longer R7.2
- net N$16: now also R7.2, R8.1; no longer R4.2, R6.1
- net N$2: now also C8.1; no longer C4.1
- net N$5: now also CB1.A; no longer CB0.A
- net N$6: now also CB0.A; no longer CB1.A
- net N$7: now also C8.2; no longer C4.2
- net N$8: now also C9.1; no longer C5.1
- net N$9: now also C9.2; no longer C5.2
- net TX_TTL: now also R4.1; no longer R7.1
- net TX_TTL_INV: now also R6.2; no longer R8.2
- net TX_TTL_MAXIM: now also R7.1; no longer R4.1
Other:
- moved on the sheet: C1, C5, R2, R3, R4, R6, R7, R8
